File: ATLabControlModule.kicad_sch (KiCad schematic)
At the start: 7 parts, among them J1 USB_Type_C_Receptacle, U1 STM32G0B1KEUx, U2 USBLC6-2P6

Commit message: update library and schematic
Parts:
- added C2: 10µ, ATLabControlModule:C_0805_(2012_Metric), symbol ATLabControlModule:C_0805_(2012_Metric)
- added C3: 100nF, ATLabControlModule:C_0402_(1005_Metric), symbol ATLabControlModule:C_0402_(1005_Metric)
- added C4: 10µF, ATLabControlModule:C_0805_(2012_Metric), symbol ATLabControlModule:C_0805_(2012_Metric)
- added D1, D2: SK6812MINI-E, ATLabControlModule:LED_SK6812MINI-E_3.2x2.8mm_P1.5mm_ReverseMount, symbol ATLabControlModule:SK6812MINI-E
- added D3, D4, D5, D6, D7: SK6805, ATLabControlModule:LED_SK6812_EC15_1.5x1.5mm, symbol ATLabControlModule:SK6805
- added J2: Conn_ARM_SWD_TagConnect_TC2030, ATLabControlModule:Tag-Connect_TC2030-IDC-NL_2x03_P1.27mm_Vertical, symbol ATLabControlModule:Conn_ARM_SWD_TagConnect_TC2030
- added R4: 10k, ATLabControlModule:R_0402_(1005_Metric), symbol ATLabControlModule:R_0402_(1005_Metric)
- added SW1, SW2: Kailh_Choc_V2_Brown, ATLabControlModule:SW_Kailh_Choc_V2, symbol ATLabControlModule:Kailh_Choc_V2_Brown
- added U3: MIC5317-3.3xM5, ATLabControlModule:SOT-23-5, symbol ATLabControlModule:MIC5317-3.3xM5
Connections:
- net GND: now also U1.33 (VSS), U1.5 (VSS), C2.2, C3.2, C4.2, D1.1 (VSS), D2.1 (VSS), D3.2 (VSS), D4.2 (VSS), D5.2 (VSS), D6.2 (VSS), D7.2 (VSS), J2.5 (GND), U3.2 (GND)
- net VBUS: now reaches J1.A4 (VBUS), J1.A9 (VBUS), J1.B4 (VBUS), J1.B9 (VBUS)
- net VBUS: now also U2.5 (VBUS), C2.1, D1.3 (VDD), D2.3 (VDD), D3.4 (VDD), D4.4 (VDD), D5.4 (VDD), D6.4 (VDD), D7.4 (VDD), R4.1, U3.1 (VIN)
- net at U2.4 (I/O2): now also U1.23 (PA10/PA12)
- net at U2.6 (I/O1): now also U1.22 (PA9/PA11)
- net at U1.18 (PA8): now also D1.2 (DIN)
- net at U1.24 (PA13): now also J2.2 (SWDIO)
- net at U1.25 (PA14): now also J2.4 (SWCLK)
- net +3V3: now reaches U1.4 (VDD)
- net +3V3: now also C4.1, J2.1 (VCC), U3.5 (VOUT)
- net at U1.6 (PF2): now also J2.3 (~{RESET})
- new net: D6.1 (DOUT), D7.3 (DIN)
- new net: D5.1 (DOUT), D6.3 (DIN)
- new net: C3.1, R4.2, U3.3 (EN)
- new net: D4.1 (DOUT), D5.3 (DIN)
- new net: D3.1 (DOUT), D4.3 (DIN)
- new net: D2.4 (DOUT), D3.3 (DIN)
- new net: D1.4 (DOUT), D2.2 (DIN)
- no-connect marks 2 -> 4
Other:
- moved on the sheet: C1, J1, R1, R2, R3, U1, U2

Commit message: schematic rev A
Parts:
- added C10, C11, C12, C13, C14, C6, C7, C8, C9: 100nF, ATLabControlModule:C_0402_(1005_Metric), symbol ATLabControlModule:C_0402_(1005_Metric)
- added C5: 10µF, ATLabControlModule:C_0805_(2012_Metric), symbol ATLabControlModule:C_0805_(2012_Metric)
- added R5: 0R, ATLabControlModule:R_0402_(1005_Metric), symbol ATLabControlModule:R_0402_(1005_Metric)
- added U4: SN74LVC1G17DBVRG4, ATLabControlModule:SOT-23-5, symbol ATLabControlModule:SN74LVC1G17DBVRG4
- renumbered SW2 to SW1, SW1 to SW2
Connections:
- net +3V3: now also C5.1, C6.1
- net GND: now also SW1.2, SW2.2, C10.2, C11.2, C12.2, C13.2, C14.2, C5.2, C6.2, C7.2, C8.2, C9.2, U4.3 (GND)
- net VBUS: now also C10.1, C11.1, C12.1, C13.1, C14.1, C7.1, C8.1, C9.1, U4.5 (VCC)
- net at SW1.1: now also U1.8 (PA1)
- net at SW2.1: now also U1.7 (PA0)
- net at D2.4 (DOUT), D3.3 (DIN): now also R5.1
- net at U1.18 (PA8): now also U4.2; no longer D1.2 (DIN)
- new net: D1.2 (DIN), R5.2, U4.4
- no-connect marks 4 -> 26
Other:
- note added: "LED Status Bar"
- note added: "START"
- note added: "STOP"
- note added: "SWD-Interface"
- company: (none) -> Tobias Netzer
- title: (none) -> ATLab Control Module
- moved on the sheet: C1, C2, C3, C4, D1, D2, D3, J1, J2, R1, R2, R3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

Commit message: PCB Rev A
Parts:
- added H1, H2, H3, H4: MountingHole, ATLabControlModule:Mounting_Hole, symbol ATLabControlModule:MountingHole
- C1, R3: now not fitted
- D1, D2: Distributor (none) -> JLCPCB; Distributor Part Number (none) -> C5149201; Manufacturer (none) -> OPSCO Optoelectronics; Manufacturer Part Number (none) -> SK6812MINI-E
- D3, D4, D5, D6, D7: Distributor (none) -> JLCPCB; Distributor Part Number (none) -> C2890035; Manufacturer (none) -> OPSCO Optoelectronics; Manufacturer Part Number (none) -> SK6805-EC15
- SW1, SW2: Distributor (none) -> Max Gaming; Distributor Part Number (none) -> 27248; Manufacturer (none) -> Kailh; Manufacturer Part Number (none) -> CPG135301D02
- U4: Distributor (none) -> Digikey; Distributor Part Number (none) -> 296-37652-1-ND; Manufacturer (none) -> Texas Instruments; Manufacturer Part Number (none) -> SN74LVC1G17DBVRG4
Connections:
- net GND: now also D3.4 (VSS), D4.4 (VSS), D5.4 (VSS), D6.4 (VSS), D7.4 (VSS); no longer D3.2 (VSS), D4.2 (VSS), D5.2 (VSS), D6.2 (VSS), D7.2 (VSS)
- net VBUS: now also D3.2 (VDD), D4.2 (VDD), D5.2 (VDD), D6.2 (VDD), D7.2 (VDD); no longer D3.4 (VDD), D4.4 (VDD), D5.4 (VDD), D6.4 (VDD), D7.4 (VDD)
- net at D4.1 (DIN): now also D3.3 (DOUT); no longer D5.3 (DIN)
- net at D4.3 (DOUT): now also D5.1 (DIN); no longer D3.1 (DOUT)
- net at D7.1 (DIN): now also D6.3 (DOUT)
- net at D7.3 (DOUT): no longer D6.1 (DOUT)
- net at D2.4 (DOUT), R5.1: now also D3.1 (DIN); no longer D3.3 (DIN)
- new net: D5.3 (DOUT), D6.1 (DIN)

Commit message: cleanup and add docs
Parts:
- U1: Distributor (none) -> Digikey; Distributor Part Number (none) -> 497-STM32G0B1KEU6-ND; Manufacturer (none) -> STMicroelectronics; Manufacturer Part Number (none) -> STM32G0B1KEU6
Changed lines of the file:
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@@
 			)
 		)
-		(property "Manufacturer" ""
+		(property "Manufacturer" "STMicroelectronics"
 			(at 165.1 137.16 0)
 			(hide yes)
@@
 			)
 		)
-		(property "Manufacturer Part Number" ""
+		(property "Manufacturer Part Number" "STM32G0B1KEU6"
 			(at 165.1 137.16 0)
 			(hide yes)
@@
 			)
 		)
-		(property "Distributor" ""
+		(property "Distributor" "Digikey"
 			(at 165.1 137.16 0)
 			(hide yes)
@@
 			)
 		)
-		(property "Distributor Part Number" ""
+		(property "Distributor Part Number" "497-STM32G0B1KEU6-ND"
 			(at 165.1 137.16 0)
 			(hide yes)
